Commit message: feat: Move laser sensor in front and lower in order to cope with low windows

File: my_robot/urdf/my_robot.xacro (robot description, xacro)
@@ -247,5 +247,5 @@
     </link>
      <joint type="fixed" name="hokuyo_joint">
-        <origin xyz="0 0.25 0.05" rpy="0 0 0"/>
+        <origin xyz="0 0.275 0" rpy="0 0 1.570796"/>
         <axis xyz="0 1 0"/>
         <parent link="crossbar_main"/>

Commit message: feat: Rotate robot for 90 grad

File: my_robot/urdf/my_robot.xacro (robot description, xacro)
@@ -2,5 +2,5 @@
 <robot name="my_robot" xmlns:xacro="http://www.ros.org/wiki/xacro">
     <xacro:include filename="$(find my_robot)/urdf/my_robot.gazebo" />
-    <link name="robot_footprint"></link>
+    <link name="robot_footprint"/>
     <link name="crossbar_main">
         <inertial>
@@ -16,5 +16,5 @@
             <origin xyz="0 0 0" rpy=" 0 0 0"/>
             <geometry>
-                <box size="0.1 0.5 0.05"/>
+                <box size="0.5 0.1 0.05"/>
             </geometry>
         </collision>
@@ -22,9 +22,9 @@
             <origin xyz="0 0 0" rpy=" 0 0 0"/>
             <geometry>
-                <box size="0.1 0.5 0.049"/>
+                <box size="0.5 0.1 0.049"/>
             </geometry>
         </visual>
         <collision name='caster_collision'>
-            <origin xyz="0 -0.25 -0.05" rpy=" 0 0 0"/>
+            <origin xyz="-0.25 0 -0.05" rpy=" 0 0 0"/>
             <geometry>
                 <sphere radius="0.049"/>
@@ -32,5 +32,5 @@
         </collision>
         <visual name='caster_visual'>
-            <origin xyz="0 -0.25 -0.05" rpy=" 0 0 0"/>
+            <origin xyz="-0.25 0 -0.05" rpy=" 0 0 0"/>
             <geometry>
                 <sphere radius="0.049"/>
@@ -38,5 +38,5 @@
         </visual>
         <collision name='caster_collision_fw'>
-            <origin xyz="0 0.24 -0.05" rpy=" 0 0 0"/>
+            <origin xyz="0.24 0 -0.05" rpy=" 0 0 0"/>
             <geometry>
                 <sphere radius="0.049"/>
@@ -44,5 +44,5 @@
         </collision>
         <visual name='caster_visual_fw'>
-            <origin xyz="0 0.20 -0.05" rpy=" 0 0 0"/>
+            <origin xyz="0.20 0 -0.05" rpy=" 0 0 0"/>
             <geometry>
                 <sphere radius="0.05"/>
@@ -51,5 +51,5 @@
     </link>
     <joint name="ctc_joint" type="fixed">
-        <origin xyz="0 0.1 0" rpy="0 0 0"/>
+        <origin xyz="0.1 0 0" rpy="0 0 0"/>
         <parent link="robot_footprint"/>
         <child link="crossbar_trans_center"/>
@@ -73,5 +73,5 @@
             <origin xyz="0 0 0" rpy=" 0 0 0"/>
             <geometry>
-                <box size="0.5 0.05 0.05"/>
+                <box size="0.05 0.5 0.05"/>
             </geometry>
         </collision>
@@ -79,10 +79,10 @@
             <origin xyz="0 0 0" rpy=" 0 0 0"/>
             <geometry>
-                <box size="0.5 0.05 0.05"/>
+                <box size="0.05 0.5 0.05"/>
             </geometry>
         </visual>
     </link>
     <joint name="ctf_joint" type="fixed">
-        <origin xyz="0 0.275 0" rpy="0 0 0"/>
+        <origin xyz="0.275 0 0" rpy="0 0 0"/>
         <parent link="robot_footprint"/>
         <child link="crossbar_trans_forward"/>
@@ -101,5 +101,5 @@
             <origin xyz="0 0 0" rpy=" 0 0 0"/>
             <geometry>
-                <box size="0.4 0.05 0.05"/>
+                <box size="0.05 0.4 0.05"/>
             </geometry>
         </collision>
@@ -107,5 +107,5 @@
             <origin xyz="0 0 0" rpy=" 0 0 0"/>
             <geometry>
-                <box size="0.4 0.05 0.05"/>
+                <box size="0.05 0.4 0.05"/>
             </geometry>
         </visual>
@@ -135,5 +135,5 @@
     </link>
     <joint name="tail_joint" type="fixed">
-        <origin xyz="0 -0.25 0.05" rpy="0 0 0"/>
+        <origin xyz="-0.25 0 0.05" rpy="0 0 0"/>
         <parent link="crossbar_main"/>
         <child link="tail"/>
@@ -144,8 +144,8 @@
                 <cylinder radius="0.1" length="0.05"/>
             </geometry>
-            <origin xyz="0 0 0" rpy="0 1.5707 0"/>
-        </collision>
-        <inertial>
-            <origin xyz="0 0 0" rpy="0 1.5707 0"/>
+            <origin xyz="0 0 0" rpy="1.5707 0 0"/>
+        </collision>
+        <inertial>
+            <origin xyz="0 0 0" rpy="1.5707 0 0"/>
             <mass value="0.5"/>
             <inertia ixx="0.1" ixy="0" ixz="0"  iyy="0.1" iyz="0" izz="0.1"/>
@@ -155,12 +155,12 @@
                 <cylinder radius="0.1" length="0.05"/>
             </geometry>
-            <origin xyz="0 0 0" rpy="0 1.5707 0"/>
+            <origin xyz="0 0 0" rpy="1.5707 0 0"/>
         </visual>
     </link>
     <joint type="continuous" name="left_wheel_hinge">
-        <origin xyz="-0.225 0 0" rpy="0 0 0"/>
+        <origin xyz="0 0.225 0" rpy="0 0 0"/>
         <child link="left_wheel"/>
         <parent link="crossbar_trans_center"/>
-        <axis xyz="-1 0 0" rpy="0 0 0"/>
+        <axis xyz="0 1 0" rpy="0 0 0"/>
         <limit effort="10000" velocity="1000"/>
         <dynamics damping="1.0" friction="1.0"/>
@@ -171,8 +171,8 @@
                 <cylinder radius="0.1" length="0.05"/>
             </geometry>
-            <origin xyz="0 0 0" rpy="0 1.5707 0"/>
-        </collision>
-        <inertial>
-            <origin xyz="0 0 0" rpy="0 1.5707 0"/>
+            <origin xyz="0 0 0" rpy="1.5707 0 0"/>
+        </collision>
+        <inertial>
+            <origin xyz="0 0 0" rpy="1.5707 0 0"/>
             <mass value="0.5"/>
             <inertia ixx="0.1" ixy="0" ixz="0"  iyy="0.1" iyz="0" izz="0.1"/>
@@ -182,12 +182,12 @@
                 <cylinder radius="0.1" length="0.05"/>
             </geometry>
-            <origin xyz="0 0 0" rpy="0 1.5707 0"/>
+            <origin xyz="0 0 0" rpy="1.5707 0 0"/>
         </visual>
     </link>
     <joint type="continuous" name="right_wheel_hinge">
-        <origin xyz="0.225 0 0" rpy="0 0 0"/>
+        <origin xyz="0 -0.225 0" rpy="0 0 0"/>
         <child link="right_wheel"/>
         <parent link="crossbar_trans_center"/>
-        <axis xyz="-1 0 0" rpy="0 0 0"/>
+        <axis xyz="0 1 0" rpy="0 0 0"/>
         <limit effort="10000" velocity="1000"/>
         <dynamics damping="1.0" friction="1.0"/>
@@ -214,6 +214,6 @@
     </link>
     <joint type="fixed" name="camera_joint">
-        <origin xyz="0 0.15 0.1" rpy="0 0 1.5707"/>
-        <axis xyz="0 1 0"/>
+        <origin xyz="0.15 0 0.1" rpy="0 0 0"/>
+        <axis xyz="1 0 0"/>
         <parent link="tail"/>
         <child link="camera"/>
@@ -222,5 +222,5 @@
     </link>
     <joint name="camera_optical_joint" type="fixed">
-        <origin xyz="0 0 0" rpy="1.5707 3.1416 0"/>
+        <origin xyz="0 0 0" rpy="-1.5707 0 -1.5707"/>
         <parent link="camera"/>
         <child link="camera_link_optical"/>
@@ -247,5 +247,5 @@
     </link>
      <joint type="fixed" name="hokuyo_joint">
-        <origin xyz="0 0.275 0" rpy="0 0 1.570796"/>
+        <origin xyz="0.275 0 0" rpy="0 0 0"/>
         <axis xyz="0 1 0"/>
         <parent link="crossbar_main"/>
@@ -264,10 +264,10 @@
         <material>Gazebo/Red</material>
     </gazebo>
+    <gazebo reference="right_wheel">
+        <material>Gazebo/Black</material>
+    </gazebo>
     <gazebo reference="left_wheel">
         <material>Gazebo/Black</material>
     </gazebo>
-    <gazebo reference="right_wheel">
-        <material>Gazebo/Black</material>
-    </gazebo>
     <gazebo reference="camera">
         <material>Gazebo/Blue</material>
